File: BidenCard.kicad_pcb (KiCad board)
At the start: 2 copper layers, 117.2 x 100 mm, 39 parts, among them J1 QL_SLOT_DIN41612_CARD, J2 Conn_02x17_Odd_Even, U1 GAL16V8, U13 FDC_WD1772, U14 27C128, U15 74HC04, U16 74LS175, U17 74ls175, U18 7805, U2 AS6C4008-55PCN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

Commit message: update PCB silkscreen for revision 2
Other:
- board text added: "Revision 2"
- board text removed: "Revision 1"
